Commit message: Created a new launch file

File: src/medibot_description/urdf/medibot.urdf (robot description, URDF)
Before this commit: robot medibot, 1 links, 0 joints
Links:
- added link laser_link
- added link left_wheel; visual cylinder length=0.05 radius=0.1
- added link right_wheel; visual cylinder length=0.05 radius=0.1
- link base_link: mass 10.0 -> None; geometry visual box size=0.5 0.3 0.2
Joints:
- added joint laser_joint: type fixed, parent base_link, child laser_link, origin xyz=0 0 0.25
- added joint left_wheel_joint: type continuous, parent base_link, child left_wheel, origin xyz=0 0.2 0, axis 0 1 0
- added joint right_wheel_joint: type continuous, parent base_link, child right_wheel, origin xyz=0 -0.2 0, axis 0 1 0
